File: sch pcb import/vectron.kicad_pcb (KiCad board)
At the start: 2 copper layers, 0 parts

Commit message: minor changes
Parts:
- added BT201: BATT_3V, Battery:BatteryHolder_Multicomp_BC-2001_1x2032_modified, F.Cu at (178.8, 137.7)
- added C201: 10uf, Capacitor_SMD:C_0603_1608Metric, F.Cu at (120.4, 149.6)
- added C202: 10uf, Capacitor_SMD:C_0603_1608Metric, F.Cu at (120.4, 152.1)
- added C203: 100nf, Capacitor_SMD:C_0603_1608Metric, F.Cu at (120.4, 154.6)
- added C204: 10uf, Capacitor_SMD:C_0603_1608Metric, F.Cu at (197.3, 134.5)
- added C205: 100nf, Capacitor_SMD:C_0603_1608Metric, F.Cu at (197.3, 137.0)
- added C206: 22uf, Capacitor_SMD:C_0603_1608Metric, F.Cu at (112.4, 153.0)
- added C207: 22uf, Capacitor_SMD:C_0603_1608Metric, F.Cu at (116.4, 140.4)
- added C208: 100nf, Capacitor_SMD:C_0603_1608Metric, F.Cu at (116.4, 142.9)
- added C209: 10uf, Capacitor_SMD:C_0603_1608Metric, F.Cu at (128.5, 98.5)
- added C210: 10uf, Capacitor_SMD:C_0603_1608Metric, F.Cu at (128.5, 102.5)
- added C211: 100nf, Capacitor_SMD:C_0603_1608Metric, F.Cu at (131.1, 118.6)
- added C212: 22uf, Capacitor_SMD:C_0603_1608Metric, F.Cu at (121.9, 95.0)
- added C213: 22uf, Capacitor_SMD:C_0603_1608Metric, F.Cu at (125.9, 82.5)
- added C214: 100nf, Capacitor_SMD:C_0603_1608Metric, F.Cu at (125.9, 85.0)
- added C215: 100nf, Capacitor_SMD:C_0603_1608Metric, F.Cu at (205.3, 132.0)
- added C216: 10uf, Capacitor_SMD:C_0603_1608Metric, F.Cu at (205.3, 134.5)
- added C217: 10uf, Capacitor_SMD:C_0603_1608Metric, F.Cu at (205.3, 137.0)
- added C218: 100nf, Capacitor_SMD:C_0603_1608Metric, F.Cu at (205.3, 139.6)
- added C301: 10uf, Capacitor_SMD:C_0603_1608Metric, F.Cu at (164.3, 90.4)
- added C302: 10uf, Capacitor_SMD:C_0603_1608Metric, F.Cu at (164.3, 92.9)
- added C303: 10uf, Capacitor_SMD:C_0603_1608Metric, F.Cu at (164.3, 95.4)
- added C304: 100nf, Capacitor_SMD:C_0603_1608Metric, F.Cu at (164.3, 97.9)
- added C305: 100nf, Capacitor_SMD:C_0603_1608Metric, F.Cu at (164.3, 100.4)
- added C306: 10uf, Capacitor_SMD:C_0603_1608Metric, F.Cu at (164.3, 103.0)
- added C307: 100nf, Capacitor_SMD:C_0603_1608Metric, F.Cu at (164.3, 105.5)
- added C308: 100nf, Capacitor_SMD:C_0603_1608Metric, F.Cu at (168.3, 90.4)
- added C309: 10uf, Capacitor_SMD:C_0603_1608Metric, F.Cu at (168.3, 92.9)
- added C310: 100nf, Capacitor_SMD:C_0603_1608Metric, F.Cu at (168.3, 95.4)
- added C311: 10uf, Capacitor_SMD:C_0603_1608Metric, F.Cu at (168.3, 97.9)
- added C312: 100nf, Capacitor_SMD:C_0603_1608Metric, F.Cu at (168.3, 100.4)
- added C313: 100nf, Capacitor_SMD:C_0603_1608Metric, F.Cu at (168.3, 103.0)
- added C401: 100nf, Capacitor_SMD:C_0603_1608Metric, F.Cu at (220.8, 48.2)
- added C402: 100nf, Capacitor_SMD:C_0603_1608Metric, F.Cu at (220.8, 50.7)
- added C403: 100nf, Capacitor_SMD:C_0603_1608Metric, F.Cu at (220.8, 53.2)
- added C404: 100nf, Capacitor_SMD:C_0603_1608Metric, F.Cu at (220.8, 55.7)
- added C405: 100nf, Capacitor_SMD:C_0603_1608Metric, F.Cu at (220.8, 58.2)
- added C406: 100nf, Capacitor_SMD:C_0603_1608Metric, F.Cu at (220.8, 60.7)
- added C407: 4u7f, Capacitor_SMD:C_0603_1608Metric, F.Cu at (220.8, 63.2)
- added C408: 220nf, Capacitor_SMD:C_0603_1608Metric, F.Cu at (224.8, 48.2)
- added C409: 100nf, Capacitor_SMD:C_0603_1608Metric, F.Cu at (224.8, 50.7)
- added C410: 100nf, Capacitor_SMD:C_0603_1608Metric, F.Cu at (224.8, 53.2)
- added C411: 100nf, Capacitor_SMD:C_0603_1608Metric, F.Cu at (224.8, 55.7)
- added C412: 2n2f, Capacitor_SMD:C_0603_1608Metric, F.Cu at (224.8, 58.2)
- added C413: 100nf, Capacitor_SMD:C_0603_1608Metric, F.Cu at (224.8, 60.7)
- added C414: 100nf, Capacitor_SMD:C_0603_1608Metric, F.Cu at (224.8, 63.2)
- added C415: 100nf, Capacitor_SMD:C_0603_1608Metric, F.Cu at (228.8, 48.2)
- added C416: 10uf, Capacitor_SMD:C_0603_1608Metric, F.Cu at (228.8, 50.7)
- added C417: 100nf, Capacitor_SMD:C_0603_1608Metric, F.Cu at (228.8, 53.2)
- added C418: 100nf, Capacitor_SMD:C_0603_1608Metric, F.Cu at (228.8, 55.7)
- added C501: 10uf, Capacitor_SMD:C_0603_1608Metric, F.Cu at (238.9, 127.5)
- added C502: 10uf, Capacitor_SMD:C_0603_1608Metric, F.Cu at (238.9, 130.0)
- added C503: 3pf, Capacitor_SMD:C_0603_1608Metric, F.Cu at (238.9, 132.5)
- added C504: 3pf, Capacitor_SMD:C_0603_1608Metric, F.Cu at (238.9, 135.1)
- added C505: 10uf, Capacitor_SMD:C_0603_1608Metric, F.Cu at (238.9, 137.6)
- added C506: 10uf, Capacitor_SMD:C_0603_1608Metric, F.Cu at (238.9, 140.1)
- added C507: 10uf, Capacitor_SMD:C_0603_1608Metric, F.Cu at (238.9, 142.6)
- added C508: 10uf, Capacitor_SMD:C_0603_1608Metric, F.Cu at (242.9, 127.5)
- added C509: 10uf, Capacitor_SMD:C_0603_1608Metric, F.Cu at (242.9, 130.0)
- added C510: 10uf, Capacitor_SMD:C_0603_1608Metric, F.Cu at (242.9, 132.5)
- added C511: 10uf, Capacitor_SMD:C_0603_1608Metric, F.Cu at (242.9, 135.1)
- added C512: 10uf, Capacitor_SMD:C_0603_1608Metric, F.Cu at (242.9, 137.6)
- added C601: 100nf, Capacitor_SMD:C_0603_1608Metric, F.Cu at (220.8, 80.9)
- added C602: 100nf, Capacitor_SMD:C_0603_1608Metric, F.Cu at (220.8, 83.4)
- added C603: 100nf, Capacitor_SMD:C_0603_1608Metric, F.Cu at (220.8, 85.9)
- added C604: 100nf, Capacitor_SMD:C_0603_1608Metric, F.Cu at (220.8, 88.4)
- added C605: 100nf, Capacitor_SMD:C_0603_1608Metric, F.Cu at (220.8, 90.9)
- added C606: 100nf, Capacitor_SMD:C_0603_1608Metric, F.Cu at (220.8, 93.4)
- added D201: SS24-SMB, Diode_SMD:D_SMB, F.Cu at (176.4, 152.0)
- added D202: white, LED_SMD:LED_0603_1608Metric, F.Cu at (182.6, 150.5)
- added D203: white, LED_SMD:LED_0603_1608Metric, F.Cu at (182.6, 153.1)
- added D301: WS2812B, LED_SMD:LED_WS2812B_PLCC4_5.0x5.0mm_P3.2mm, F.Cu at (212.7, 102.4)
- added D302: blue, LED_SMD:LED_0603_1608Metric, F.Cu at (213.4, 68.1)
- added D303: blue, LED_SMD:LED_0603_1608Metric, F.Cu at (213.4, 70.7)
- added D304: blue, LED_SMD:LED_0603_1608Metric, F.Cu at (213.4, 73.3)
- added D401: SS24-SMB, LED_SMD:LED_0603_1608Metric, F.Cu at (246.4, 58.9)
- added D501: green, LED_SMD:LED_0603_1608Metric, F.Cu at (260.6, 138.7)
- added D601: red, LED_SMD:LED_0603_1608Metric, F.Cu at (232.8, 87.5)
- added D602: red, LED_SMD:LED_0603_1608Metric, F.Cu at (232.8, 90.1)
- added H101: MountingHole_Pad, MountingHole:MountingHole_2.2mm_M2_Pad_Via, F.Cu at (277.4, 84.7)
- added H102: MountingHole_Pad, MountingHole:MountingHole_2.2mm_M2_Pad_Via, F.Cu at (277.4, 90.7)
- added H103: MountingHole_Pad, MountingHole:MountingHole_2.2mm_M2_Pad_Via, F.Cu at (277.4, 96.6)
- added H104: MountingHole_Pad, MountingHole:MountingHole_2.2mm_M2_Pad_Via, F.Cu at (277.4, 102.6)
- added J201: XT30PW-M, XT30PW-M:AMASS_XT30PW-M, F.Cu at (202.7, 112.4)
- added J202: Screw_01x02, TerminalBlock:TerminalBlock_Xinya_XY308-2.54-2P_1x02_P2.54mm_Horizontal, F.Cu at (210.2, 144.9)
- added J301: USB_C_Receptacle_USB2.0_16P, Connector_USB:USB_C_Receptacle_GCT_USB4105-xx-A_16P_TopMnt_Horizontal, F.Cu at (206.0, 94.4)
- added J302: Conn_01x04_Pin, Connector_PinHeader_2.54mm:PinHeader_1x04_P2.54mm_Vertical, F.Cu at (180.6, 91.4)
- added J501: Conn_Coaxial, Connector_Coaxial:SMA_Amphenol_901-143_Horizontal, F.Cu at (253.7, 138.8)
- added J502: 0734120114, digikey-footprints:Molex_734120114_UMC_RF_CONN_Vertical, F.Cu at (261.4, 129.0)
- added J503: 0734120114, digikey-footprints:Molex_734120114_UMC_RF_CONN_Vertical, F.Cu at (261.4, 134.6)
- added J504: Micro_SD_Card, Connector_Card:microSD_HC_Molex_47219-2001, F.Cu at (225.7, 143.1)
- added J505: Screw_Terminal_01x06, TerminalBlock:TerminalBlock_Xinya_XY308-2.54-6P_1x06_P2.54mm_Horizontal, F.Cu at (219.9, 130.4)
- added J601: Screw_Terminal_01x04, TerminalBlock:TerminalBlock_Xinya_XY308-2.54-4P_1x04_P2.54mm_Horizontal, F.Cu at (221.3, 98.8)
- added JP301: Jumper, Jumper:SolderJumper-2_P1.3mm_Open_RoundedPad1.0x1.5mm, F.Cu at (213.5, 48.7)
- added JP302: Jumper, Jumper:SolderJumper-2_P1.3mm_Open_RoundedPad1.0x1.5mm, F.Cu at (213.5, 52.2)
- added JP303: Jumper, Jumper:SolderJumper-2_P1.3mm_Open_RoundedPad1.0x1.5mm, F.Cu at (213.5, 55.8)
- added JP401: Jumper, Jumper:SolderJumper-2_P1.3mm_Open_RoundedPad1.0x1.5mm, F.Cu at (237.0, 48.7)
- added JP402: Jumper, Jumper:SolderJumper-2_P1.3mm_Open_RoundedPad1.0x1.5mm, F.Cu at (237.0, 52.2)
- added JP403: Jumper, Jumper:SolderJumper-2_P1.3mm_Open_RoundedPad1.0x1.5mm, F.Cu at (237.0, 55.8)
- added JP404: Jumper, Jumper:SolderJumper-2_P1.3mm_Open_RoundedPad1.0x1.5mm, F.Cu at (237.0, 59.3)
- added L201: SWPA5040S3R3NT 3u3h, Inductor_SMD:L_Sunlord_SWPA5040S, F.Cu at (100.1, 162.7)
- added L202: SWPA5040S3R3NT 3u3h, Inductor_SMD:L_Sunlord_SWPA5040S, F.Cu at (105.7, 111.4)
- added L501: 10nh, Inductor_SMD:L_0402_1005Metric, F.Cu at (250.3, 144.6)
- added L502: 27nh, Inductor_SMD:L_0402_1005Metric, F.Cu at (250.3, 146.6)
- added LS401: CMT-8530S-SMT, CMT-8530S-SMT:CUI_CMT-8530S-SMT, F.Cu at (224.3, 70.0)
- added Q301: SS8050, Package_TO_SOT_SMD:SOT-23-3, F.Cu at (213.9, 59.9)
- added Q302: SS8050, Package_TO_SOT_SMD:SOT-23-3, F.Cu at (213.9, 64.6)
- added Q401: SS8050, Package_TO_SOT_SMD:SOT-23-3, F.Cu at (241.7, 55.6)
- added Q601: SISA12ADN, Package_SO:Vishay_PowerPAK_1212-8_Single, F.Cu at (234.4, 97.1)
- added Q602: SISA12ADN, Package_SO:Vishay_PowerPAK_1212-8_Single, F.Cu at (234.4, 101.8)
- added R201: 18k, Resistor_SMD:R_0603_1608Metric, F.Cu at (209.3, 127.0)
- added R202: 18k, Resistor_SMD:R_0603_1608Metric, F.Cu at (209.3, 129.5)
- added R203: 4k7, Resistor_SMD:R_0603_1608Metric, F.Cu at (132.4, 154.6)
- added R204: 10k, Resistor_SMD:R_0603_1608Metric, F.Cu at (209.3, 134.5)
- added R205: 10k, Resistor_SMD:R_0603_1608Metric, F.Cu at (209.3, 137.0)
- added R206: 54k9, Resistor_SMD:R_0603_1608Metric, F.Cu at (132.4, 162.1)
- added R207: 10k, Resistor_SMD:R_0603_1608Metric, F.Cu at (136.5, 149.6)
- added R208: 4k7, Resistor_SMD:R_0603_1608Metric, F.Cu at (143.5, 96.3)
- added R209: 33k2, Resistor_SMD:R_0603_1608Metric, F.Cu at (143.5, 98.8)
- added R210: 10k, Resistor_SMD:R_0603_1608Metric, F.Cu at (143.5, 101.3)
- added R211: 1k, Resistor_SMD:R_0603_1608Metric, F.Cu at (213.3, 137.0)
- added R212: 1k, Resistor_SMD:R_0603_1608Metric, F.Cu at (213.3, 139.6)
- added R301: 10k, Resistor_SMD:R_0603_1608Metric, F.Cu at (168.3, 105.5)
- added R302: 4k7, Resistor_SMD:R_0603_1608Metric, F.Cu at (172.3, 90.4)
- added R303: 4k7, Resistor_SMD:R_0603_1608Metric, F.Cu at (172.3, 92.9)
- added R304: 10k, Resistor_SMD:R_0603_1608Metric, F.Cu at (172.3, 95.4)
- added R305: 1k, Resistor_SMD:R_0603_1608Metric, F.Cu at (172.3, 97.9)
- added R306: 1k, Resistor_SMD:R_0603_1608Metric, F.Cu at (172.3, 100.4)
- added R307: 2k2, Resistor_SMD:R_0603_1608Metric, F.Cu at (172.3, 103.0)
- added R308: 2k2, Resistor_SMD:R_0603_1608Metric, F.Cu at (172.3, 105.5)
- added R309: 1k, Resistor_SMD:R_0603_1608Metric, F.Cu at (176.3, 90.4)
- added R310: 10k, Resistor_SMD:R_0603_1608Metric, F.Cu at (176.3, 92.9)
- added R311: 10k, Resistor_SMD:R_0603_1608Metric, F.Cu at (176.3, 95.4)
- added R312: 5k1, Resistor_SMD:R_0603_1608Metric, F.Cu at (176.3, 97.9)
- added R313: 5k1, Resistor_SMD:R_0603_1608Metric, F.Cu at (176.3, 100.4)
- added R314: 100k, Resistor_SMD:R_0603_1608Metric, F.Cu at (176.3, 103.0)
- added R401: 10k, Resistor_SMD:R_0603_1608Metric, F.Cu at (228.8, 58.2)
- added R402: 10k, Resistor_SMD:R_0603_1608Metric, F.Cu at (228.8, 60.7)
- added R403: 10k, Resistor_SMD:R_0603_1608Metric, F.Cu at (228.8, 63.2)
- added R404: 10k, Resistor_SMD:R_0603_1608Metric, F.Cu at (232.8, 48.2)
- added R405: 1k, Resistor_SMD:R_0603_1608Metric, F.Cu at (232.8, 50.7)
- added R406: 10k, Resistor_SMD:R_0603_1608Metric, F.Cu at (232.8, 53.2)
- added R407: 10k, Resistor_SMD:R_0603_1608Metric, F.Cu at (232.8, 55.7)
- added R408: 10k, Resistor_SMD:R_0603_1608Metric, F.Cu at (232.8, 58.2)
- added R501: 10, Resistor_SMD:R_0603_1608Metric, F.Cu at (242.9, 140.1)
- added R502: 1k, Resistor_SMD:R_0603_1608Metric, F.Cu at (242.9, 142.6)
- added R503: 10k, Resistor_SMD:R_0603_1608Metric, F.Cu at (246.9, 127.5)
- added R504: 10k, Resistor_SMD:R_0603_1608Metric, F.Cu at (246.9, 130.0)
- added R505: 10k, Resistor_SMD:R_0603_1608Metric, F.Cu at (246.9, 132.5)
- added R506: 10k, Resistor_SMD:R_0603_1608Metric, F.Cu at (246.9, 135.1)
- added R507: 10k, Resistor_SMD:R_0603_1608Metric, F.Cu at (246.9, 137.6)
- added R508: 10k, Resistor_SMD:R_0603_1608Metric, F.Cu at (246.9, 140.1)
- added R509: 10k, Resistor_SMD:R_0603_1608Metric, F.Cu at (246.9, 142.6)
- added R601: 1k, Resistor_SMD:R_0603_1608Metric, F.Cu at (224.8, 80.9)
- added R602: 1k, Resistor_SMD:R_0603_1608Metric, F.Cu at (224.8, 83.4)
- added R604: 1k, Resistor_SMD:R_0603_1608Metric, F.Cu at (224.8, 85.9)
- added R605: 1k, Resistor_SMD:R_0603_1608Metric, F.Cu at (224.8, 88.4)
- added R606: 1k, Resistor_SMD:R_0603_1608Metric, F.Cu at (224.8, 90.9)
- added R607: 1k, Resistor_SMD:R_0603_1608Metric, F.Cu at (224.8, 93.4)
- added R608: 1k, Resistor_SMD:R_0603_1608Metric, F.Cu at (228.8, 80.9)
- added R610: 1k, Resistor_SMD:R_0603_1608Metric, F.Cu at (228.8, 83.4)
- added R611: 1k, Resistor_SMD:R_0603_1608Metric, F.Cu at (228.8, 85.9)
- added R612: 1k, Resistor_SMD:R_0603_1608Metric, F.Cu at (228.8, 91.2)
- added S301: TK-066S, digikey-footprints:Switch_Tactile_SMD_4.5x4.5mm_TL3315NF160Q, F.Cu at (185.3, 46.9)
- added S302: TK-066S, digikey-footprints:Switch_Tactile_SMD_4.5x4.5mm_TL3315NF160Q, F.Cu at (185.6, 55.7)
- added U201: TPS563201DDCR, TPS563201DDCR:SOT95P280X110-6N, F.Cu at (121.2, 166.3)
- added U202: TPS563201DDCR, TPS563201DDCR:SOT95P280X110-6N, F.Cu at (130.8, 113.5)
- added U203: AMS1117-3.3, Package_TO_SOT_SMD:SOT-223-3_TabPin2, F.Cu at (167.2, 153.4)
- added U301: FT232RL, Package_SO:SSOP-28_5.3x10.2mm_P0.65mm, F.Cu at (194.9, 95.2)
- added U302: ESP32-S3-WROOM-1, RF_Module:ESP32-S3-WROOM-1, F.Cu at (142.8, 50.1)
- added U303: USB6B1RL, Package_SO:SO-8_3.9x4.9mm_P1.27mm, F.Cu at (204.4, 102.5)
- added U401: BMP280, Package_LGA:Bosch_LGA-8_2x2.5mm_P0.65mm_ClockwisePinNumbering, F.Cu at (232.1, 66.5)
- added U402: BMP280, Package_LGA:Bosch_LGA-8_2x2.5mm_P0.65mm_ClockwisePinNumbering, F.Cu at (232.1, 70.3)
- added U403: BME280, Package_LGA:Bosch_LGA-8_2.5x2.5mm_P0.65mm_ClockwisePinNumbering, F.Cu at (246.6, 55.5)
- added U404: HMC5883L-TR, HMC5883L-TR:XDCR_HMC5883L-TR, F.Cu at (248.4, 75.9)
- added U405: MPU-6050, Sensor_Motion:InvenSense_QFN-24_4x4mm_P0.5mm, F.Cu at (242.3, 50.1)
- added U406: MMC5983MA, MMC5983MA:PQFN50P300X300X100-16N, F.Cu at (237.5, 75.3)
- added U407: DS3231M, Package_SO:SOIC-16W_7.5x10.3mm_P1.27mm, F.Cu at (241.3, 67.1)
- added U408: LSM6DSL, Package_LGA:LGA-14_3x2.5mm_P0.5mm_LayoutBorder3x4y, F.Cu at (232.1, 74.2)
- added U501: RFM98W-433S2, RF_Module:HOPERF_RFM9XW_SMD, F.Cu at (227.1, 117.5)
- added U502: NEO-6M-GPS, NEO-6M-GPS:XCVR_NEO-6M-GPS, F.Cu at (245.2, 117.5)
- added U503: W25Q128JVS, Package_SO:SOIC-8_5.3x5.3mm_P1.27mm, F.Cu at (242.0, 147.3)
- added U601: LM358, Package_SO:SOIC-8_3.9x4.9mm_P1.27mm, F.Cu at (235.0, 83.0)
