File: sch pcb import/vectron.kicad_pcb (KiCad board)
At the start: 2 copper layers, 183 parts, among them J201 XT30PW-M, J202 Screw_01x02, J301 USB_C_Receptacle_USB2.0_16P, J302 Conn_01x04_Pin, J501 Conn_Coaxial, J502 0734120114, J503 0734120114, J504 Micro_SD_Card, J505 Screw_Terminal_01x06, J601 Screw_Terminal_01x04, Q301 SS8050, Q302 SS8050, Q401 SS8050, Q601 SISA12ADN, Q602 SISA12ADN, U201 TPS563201DDCR, U202 TPS563201DDCR, U203 AMS1117-3.3, U301 FT232RL, U302 ESP32-S3-WROOM-1, U303 USB6B1RL, U401 BMP280, U402 BMP280, U403 BME280, U404 HMC5883L-TR, U405 MPU-6050, U406 MMC5983MA, U407 DS3231M, U408 LSM6DSL, U501 RFM98W-433S2, U502 NEO-6M-GPS, U503 W25Q128JVS, U601 LM358

Commit message: minor changes
Parts:
- removed R611, R612: 1k, Resistor_SMD:R_0603_1608Metric
- added C219: 10uf, Capacitor_SMD:C_0603_1608Metric, F.Cu at (115.3, 106.6)
- added C220: 100nf, Capacitor_SMD:C_0603_1608Metric, F.Cu at (115.3, 109.1)
- added R603: 1k, Resistor_SMD:R_0603_1608Metric, F.Cu at (190.4, 104.5)
- added R609: 1k, Resistor_SMD:R_0603_1608Metric, F.Cu at (190.4, 107.0)
- C201, C204, C209, C210, C216, C217: value 10uf -> 100nf
- C203, C205, C211, C218: value 100nf -> 10uf
- C206, C213: value 22uf -> 100nf
- C208, C214, C215: value 100nf -> 22uf
- C212: value 22uf -> 10uf
- C503, C504: value 3pf -> 10uf
- C505, C506: value 10uf -> 3pf
- J504: value Micro_SD_Card -> Screw_Terminal_01x06; footprint Connector_Card:microSD_HC_Molex_47219-2001 -> TerminalBlock:TerminalBlock_Xinya_XY308-2.54-6P_1x06_P2.54mm_Horizontal
- J505: value Screw_Terminal_01x06 -> Micro_SD_Card; footprint TerminalBlock:TerminalBlock_Xinya_XY308-2.54-6P_1x06_P2.54mm_Horizontal -> Connector_Card:microSD_HC_Molex_47219-2001
- moved C216 144.5 mm to (63.5, 162.2), turned to -90 degrees
- moved C215 143.3 mm to (65.2, 162.2), turned to -90 degrees
- moved C204 121.1 mm to (78.5, 158.4)
- moved R209 104.7 mm to (56.0, 156.3), turned to -90 degrees
- moved R210 101.7 mm to (56.0, 153.2), turned to -90 degrees
- moved R208 101.0 mm to (59.9, 153.0), turned to 180 degrees
- moved C213 100.9 mm to (59.6, 158.5)
- moved C214 97.2 mm to (66.8, 162.2), turned to -90 degrees
- moved U202 82.8 mm to (59.6, 155.7)
- moved C210 81.0 mm to (64.6, 152.3), turned to 90 degrees
- moved C212 79.8 mm to (66.3, 152.3), turned to 90 degrees
- moved C209 78.0 mm to (82.4, 161.4), turned to -90 degrees
- moved C211 76.0 mm to (63.0, 152.3), turned to 90 degrees
- moved R207 61.5 mm to (75.1, 153.3), turned to -90 degrees
- moved L202 61.0 mm to (65.2, 157.1), turned to -90 degrees
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Connections:
- C203 pad 1: /power/VBST1 -> +BATT
- C203 pad 2: /power/SW1 -> GND
- C204 pad 1: +BATT -> /power/VBST1
- C204 pad 2: GND -> /power/SW1
- C206 pad 1: +5V -> +BATT
- C209 pad 1: +BATT -> +5V
- C211 pad 1: /power/VBST2 -> +BATT
- C211 pad 2: /power/SW2 -> GND
- C212 pad 1: +3V3 -> +BATT
- C213 pad 1: +3V3 -> /power/VBST2
- C213 pad 2: GND -> /power/SW2
- C215 pad 1: +BATT -> +3V3
- C216 pad 1: +BATT -> +3V3
- C217 pad 1: +3V3 -> +BATT
- C218 pad 1: +3V3 -> +BATT
- C501 pad 1: +3V3 -> +5V
- C502 pad 1: +3V3 -> +5V
- C503 pad 1: LORA_ANT -> +3V3
- C504 pad 1: /sensors2/lora_ant_out -> +3V3
- C505 pad 1: +3V3 -> LORA_ANT
- C506 pad 1: +3V3 -> /sensors2/lora_ant_out
- C511 pad 1: +5V -> +3V3
- C512 pad 1: +5V -> +3V3
- J504 pad 1: /sensors2/dat2 -> +5V
- J504 pad 2: SD_CS -> GND
- J504 pad 3: SPI_MOSI -> SERVO1
- J504 pad 4: +3V3 -> +5V
- J504 pad 5: SPI_CLK -> GND
- J504 pad 6: GND -> SERVO2
- J505 pad 1: +5V -> /sensors2/dat2
- J505 pad 2: GND -> SD_CS
- J505 pad 3: SERVO1 -> SPI_MOSI
- J505 pad 4: +5V -> +3V3
- J505 pad 5: GND -> SPI_CLK
- J505 pad 6: SERVO2 -> GND
- R604 pad 1: /pyro/opout1 -> DRAIN1
- R604 pad 2: /pyro/opled1 -> /pyro/-opamp1
- R605 pad 1: DRAIN1 -> TRIGGER1
- R605 pad 2: /pyro/-opamp1 -> GND
- R606 pad 1: TRIGGER1 -> +3V3
- R606 pad 2: GND -> /pyro/+opamp2
- R607 pad 1: +3V3 -> /pyro/opout2
- R607 pad 2: /pyro/+opamp2 -> CONTINUITY2
- R608 pad 2: CONTINUITY2 -> /pyro/opled2
- R610 pad 1: /pyro/opout2 -> TRIGGER2
- R610 pad 2: /pyro/opled2 -> GND
Routing:
- net +5V: track 0.00 -> 10.2 mm
- net /power/SW2: track 0.00 -> 6.16 mm
- net /power/SW1: track 0.00 -> 6.16 mm
- net /power/VFB2: track 0.00 -> 3.94 mm
- net /power/EN2: track 0.00 -> 3.88 mm
- net /power/VFB1: track 0.00 -> 3.72 mm
- net /power/EN1: track 0.00 -> 3.68 mm
- net /power/VBST2: track 0.00 -> 2.04 mm
- net /power/VBST1: track 0.00 -> 1.92 mm
- added copper zone on F.Cu, net +5V
- added copper zone on F.Cu, net +BATT
- added copper zone on F.Cu, net /power/SW1
- added copper zone on F.Cu, net /power/SW2
Other:
- board outline added: 271.7 x 162.9 mm

Commit message: minor changes
Parts:
- removed C501, C502: 10uf, Capacitor_SMD:C_0603_1608Metric
- C301: value 10uf -> 100nf
- S301, S302: footprint digikey-footprints:Switch_Tactile_SMD_4.5x4.5mm_TL3315NF160Q -> Tact switch:tact switch 3.4x2.5mm
- moved U401 266.0 mm to (-18.5, -22.7)
- moved JP401 262.8 mm to (-16.6, -20.2), turned to 180 degrees
- moved R403 261.9 mm to (-18.4, -23.4)
- moved R401 259.9 mm to (-18.4, -22.0)
- moved C401 251.8 mm to (-20.8, -22.7), turned to 90 degrees
- moved C402 250.8 mm to (-19.8, -20.2), turned to 180 degrees
- moved U403 233.8 mm to (27.5, -26.1)
- moved U402 229.1 mm to (24.3, -26.0)
- moved JP402 224.1 mm to (25.9, -23.1)
- moved R402 220.1 mm to (26.2, -25.1)
- moved R404 219.8 mm to (26.2, -26.7)
- moved C403 214.1 mm to (21.8, -26.0), turned to 90 degrees
- moved C404 213.5 mm to (22.5, -23.5), turned to 180 degrees
- moved U405 181.8 mm to (76.8, -25.3)
- moved JP403 179.7 mm to (74.7, -21.3), turned to 180 degrees
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Connections:
- C601 pad 1: +3V3 -> /pyro/+opamp1
- C604 pad 1: +3V3 -> /pyro/+opamp2
- J302 pad 1: USBD- -> USBD+
- J302 pad 2: USBD+ -> USBD-
- J601 pad 2: DRAIN2 -> DRAIN1
- J601 pad 4: DRAIN1 -> DRAIN2
- Q401 pad 2: /sensors1/BUZZER_NEGATIVE -> GND
- Q401 pad 3: GND -> /sensors1/BUZZER_NEGATIVE
- R601 pad 1: +3V3 -> /pyro/+opamp1
- R601 pad 2: /pyro/+opamp1 -> +3V3
- R606 pad 1: +3V3 -> /pyro/+opamp2
- R606 pad 2: /pyro/+opamp2 -> +3V3
Routing:
- net +5V: track 10.2 -> 0.00 mm
- net RF_IN: track 0.00 -> 9.98 mm
- net /power/SW2: track 6.16 -> 0.00 mm
- net /power/SW1: track 6.16 -> 0.00 mm
- net /power/VFB2: track 3.94 -> 0.00 mm
- net /power/EN2: track 3.88 -> 0.00 mm
- net /power/VFB1: track 3.72 -> 0.00 mm
- net /power/EN1: track 3.68 -> 0.00 mm
- net /sensors2/gps_inductor: track 0.00 -> 3.35 mm
- net /sensors2/gps_pulse: track 0.00 -> 3.02 mm
- net VCC_RF: track 0.00 -> 2.89 mm
- net /power/VBST2: track 2.04 -> 0.00 mm
- net /power/VBST1: track 1.92 -> 0.00 mm
- net /sensors2/gps_led: track 0.00 -> 1.44 mm
- removed copper zone on F.Cu, net +5V
- removed copper zone on F.Cu, net +BATT
- removed copper zone on F.Cu, net /power/SW1
- removed copper zone on F.Cu, net /power/SW2
Other:
- board size 271.7 x 162.9 mm -> 80.1 x 73.3 mm
- copper layers 2 -> 4
