File: sch pcb import/power.kicad_sch (KiCad schematic)
At the start: 42 parts, among them J201 XT30PW-M, J202 Screw_01x02, U201 TPS563201DDCR, U202 TPS563201DDCR, U203 AMS1117-3.3

Commit message: added servo and finished esp32 connections
Other:
- note added: "SUPPLEMENTARY BATTERIES"
- company: Done by :- Arudhran -> Drawn by :- Arudhran
- title: AVIONICS PCB -> VECTRON
Changed lines of the file:
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@@
 	(paper "A4")
 	(title_block
-		(title "AVIONICS PCB")
-		(date "2025-05-27")
+		(title "VECTRON")
+		(date "2025-06-10")
 		(rev "1.0.0")
-		(company "Done by :- Arudhran")
+		(company "Drawn by :- Arudhran")
 	)
 	(rectangle
@@
 		)
 	)
-	(text "XT30 connector\n"
+	(text "SUPPLEMENTARY BATTERIES"
 		(exclude_from_sim no)
-		(at 85.852 46.99 0)
+		(at 84.582 47.752 0)
 		(effects
 			(font
@@
 	)
 	(global_label "PYRO_BAT"
-		(shape input)
+		(shape output)
 		(at 146.05 29.21 180)
 		(fields_autoplaced yes)
@@
 	)
 	(global_label "MAIN_BAT"
-		(shape input)
+		(shape output)
 		(at 121.92 29.21 180)
 		(fields_autoplaced yes)

Commit message: minor changes
Other:
- title: VECTRON -> VECTRON-V1
Changed lines of the file:
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@@
 	(paper "A4")
 	(title_block
-		(title "VECTRON")
-		(date "2025-06-10")
+		(title "VECTRON-V1")
+		(date "2025-06-13")
 		(rev "1.0.0")
 		(company "Drawn by :- Arudhran")

Commit message: minor changes
Parts:
- removed NT201: NetTie_2, symbol Device:NetTie_2
- BT201: footprint (none) -> Battery:BatteryHolder_Multicomp_BC-2001_1x2032_modified
- C201, C202, C203, C204, C205, C206, C207, C208, C209, C210, C211, C212, C213, C214, C215, C216, C217, C218: footprint (none) -> Capacitor_SMD:C_0603_1608Metric
- D201: footprint (none) -> Diode_SMD:D_SMB
- D202, D203: footprint (none) -> LED_SMD:LED_0603_1608Metric
- J202: footprint (none) -> TerminalBlock:TerminalBlock_Xinya_XY308-2.54-2P_1x02_P2.54mm_Horizontal
- L201, L202: footprint (none) -> Inductor_SMD:L_Sunlord_SWPA5040S
- R201, R202, R203, R204, R205, R206, R207, R208, R209, R210, R211, R212: footprint (none) -> Resistor_SMD:R_0603_1608Metric
Connections:
- net VCOM is gone; now on net +BATT: C201.1, C202.1, C209.1, C210.1, C215.1, C216.1, R203.1, R208.1, U201.3 (VIN), U202.3 (VIN), U203.3 (VI)

Commit message: minor changes
Parts:
- removed C209: 10uf, Capacitor_SMD:C_0603_1608Metric, symbol Device:C
- removed C213: 22uf, Capacitor_SMD:C_0603_1608Metric, symbol Device:C
- added C201, C216: 100nf, Capacitor_SMD:C_0603_1608Metric, symbol Device:C
- added C211: 10uf, Capacitor_SMD:C_0603_1608Metric, symbol Device:C
- added C215: 22uf, Capacitor_SMD:C_0603_1608Metric, symbol Device:C
- C210: value 10uf -> 100nf
- C212: value 22uf -> 10uf
- C214: value 100nf -> 22uf
- renumbered C201 to C202, C202 to C203, C203 to C204, C204 to C205, C205 to C206, C206 to C207, C207 to C208, C208 to C209, C211 to C213, C215 to C217, C216 to C218, C217 to C219, C218 to C220
Connections:
- net +3V3: now also C215.1, C216.1; no longer C212.1
- net +BATT: now also C212.1, C201.1, C211.1
- net GND: now also C201.2, C211.2, C215.2, C216.2
Other:
- moved on the sheet: C202, C203, C204, C207, C208, C213, L201, L202, R203, R206, R207, R208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

Commit message: minor changes
Other:
- company: Drawn by :- Arudhran -> (none)
