File: sch pcb import/vectron.kicad_sch (KiCad schematic)
At the start: 4 parts

Commit message: added servo and finished esp32 connections
Other:
- company: Done by :- Arudhran -> Drawn by :- Arudhran
- title: AVIONICS PCB -> VECTRON
Changed lines of the file:
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@@
 	(paper "A4")
 	(title_block
-		(title "AVIONICS PCB")
-		(date "2025-05-27")
+		(title "VECTRON")
+		(date "2025-06-10")
 		(rev "1.0.0")
-		(company "Done by :- Arudhran")
+		(company "Drawn by :- Arudhran")
 	)
 	(junction
@@
 		)
 		(instances
-			(project "avionics PCB"
+			(project "vectron"
 				(path "/b25900d5-7cd1-4497-821f-c15efd65d19e"
 					(page "2")
@@
 		)
 		(instances
-			(project "avionics PCB"
+			(project "vectron"
 				(path "/b25900d5-7cd1-4497-821f-c15efd65d19e"
 					(page "3")
@@
 		)
 		(instances
-			(project "avionics PCB"
+			(project "vectron"
 				(path "/b25900d5-7cd1-4497-821f-c15efd65d19e"
 					(page "5")
@@
 		)
 		(instances
-			(project "avionics PCB"
+			(project "vectron"
 				(path "/b25900d5-7cd1-4497-821f-c15efd65d19e"
 					(page "6")
@@
 		)
 		(instances
-			(project "avionics PCB"
+			(project "vectron"
 				(path "/b25900d5-7cd1-4497-821f-c15efd65d19e"
 					(page "4")

Commit message: minor changes
Other:
- title: VECTRON -> VECTRON-V1
Changed lines of the file:
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@@
 	(paper "A4")
 	(title_block
-		(title "VECTRON")
-		(date "2025-06-10")
+		(title "VECTRON-V1")
+		(date "2025-06-13")
 		(rev "1.0.0")
 		(company "Drawn by :- Arudhran")

Commit message: minor changes
Changed lines of the file:
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@@
 	)
 	(sheet
-		(at 17.78 16.51)
+		(at 16.51 16.51)
 		(size 63.5 36.83)
 		(exclude_from_sim no)
@@
 		)
 		(property "Sheetname" "power"
-			(at 17.78 15.7984 0)
+			(at 16.51 15.7984 0)
 			(effects
 				(font
@@
 		)
 		(property "Sheetfile" "power.kicad_sch"
-			(at 17.78 53.9246 0)
+			(at 16.51 53.9246 0)
 			(effects
 				(font
@@
 	(sheet
 		(at 185.42 16.51)
-		(size 60.96 38.1)
+		(size 60.96 36.83)
 		(exclude_from_sim no)
 		(in_bom yes)
@@
 		)
 		(property "Sheetfile" "sensors2.kicad_sch"
-			(at 185.42 55.1946 0)
+			(at 185.42 53.9246 0)
 			(effects
 				(font
@@
 	)
 	(sheet
-		(at 17.78 78.74)
+		(at 16.51 78.74)
 		(size 63.5 39.37)
 		(exclude_from_sim no)
@@
 		)
 		(property "Sheetname" "pyro"
-			(at 17.78 78.0284 0)
+			(at 16.51 78.0284 0)
 			(effects
 				(font
@@
 		)
 		(property "Sheetfile" "pyro.kicad_sch"
-			(at 17.78 118.6946 0)
+			(at 16.51 118.6946 0)
 			(effects
 				(font

Commit message: minor changes
Other:
- company: Drawn by :- Arudhran -> (none)
Changed lines of the file:
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@@
 		(date "2025-06-13")
 		(rev "1.0.0")
-		(company "Drawn by :- Arudhran")
+		(comment 9 "ARUDHRAN")
 	)
 	(junction
@@
 	)
 	(embedded_fonts no)
+	(embedded_files
+		(file
+			(name "drawnby.kicad_wks")
+			(type worksheet)
+			(data |KLUv/WCjCkUWAFafYyEA1w4WHCSqx1mCzrBErr1UFAnx+4M2IpX8cEv+/3+oJwJZAFMAXgAlaL7o
+				uTz/zxA9/+PBudo2sSeDJec7Thoya9X+/IhJbmLSkFm2/YTTL/kXAICAABW9p9XaKk6FR+eQaNX5
+				fDC76R6DZq29br1tnjjNPioAAoI0ROKMoIhDhW050826hmFY7VUAvHl2bGe30xOtbNVf8g8/q1d2
+				u2amUhZN/KCjnrOb+RSf7Nq1CoknGbaTj7/98z2aojODXfWbXpanePv2aDp2dbW2P4OfVlV77p/L
+				4JAajF7VD5b57HR2FKxYugpX8RO+jOQZNna9TGcZuUXTqoZYC+ut2gnFu1i6DKfBMTwIipBZWVdr
+				NwvRCS3VfVyD02EuFw9FaIU/2Mg5m7K/6WKbOvhTESi7AQGB4d5bN23TEpiV2b6uzEJgWys2i55o
+				OMtF3Gy77oXd7bKIWy/7TTqJyQTR8mTUu5lwFQmFkXh8XOXrusdF0y4Lk3CTLuI5sEPEJPi4E1a1
+				XeTzPvLxd+21I+4PgIqg8UyGmJESKUiSFDpwRKTmqhvOw4aWBWZRQuAujZYrbLBQBQHATYc2Zfm3
+				Eo69zsd5liNStkM9Tr1MhlS/W8LW8L5iQQKDMdPTt0yWQ4NkhE0+LovsXoZ8So5BbrB4EF4SOl0e
+				khTCzDE+O3mysrN5ITnRDvz5rvxhAj6UmT2EKMQka9gSgH4Ehj7fneXic/aVZ40QEOhTp3yZIFgQ
+				j4qCmKgczYBrl1INk1Xj1EF8QP+UyTFpKQeZ6VP2oIYBDX3qQasgzU8ue8p9ZLVJlxr9QYIQ3SH1
+				olHZK2dxQG6f5ThsBMg0wiItOv61V+bba3i0CwJCWiUxNbDpCxfykGD+6CZ1SsPLtuhh/mrQcMBh
+				Fo2WO1t0kNa2abmYkaJnfsZeo1eTmqZjZ/0bhou4jZw0IB2DXgU=|
+			)
+			(checksum "7B2771A299185B03AD1E56A709A1FEF8")
+		)
+	)
 )
